File: pcb/ultrasonic_microphone.kicad_pcb (KiCad board)
At the start: 4 copper layers, 30.5 x 50.8 mm, 33 parts, among them J1 Conn_01x19, J2 Conn_01x19, J3 Electret Microphone, U1 LTC6910-2CTS8-TRMPBF, U2 ADA4528-2ARMZ, U3 LTC6655CHMS8-3-PBF, U4 ADM7160ACPZN2.5-R7, U5 LTC2508CDKD-32

Commit message: Fabbed board
Parts:
- removed the C12 at (144.8, 37.1)
- removed the C13 at (139.7, 53.3)
- removed the C14 at (149.8, 55.9)
- removed the C15 at (134.6, 40.6)
- removed the C17 at (147.3, 39.6)
- removed R6, R7: 10, Resistor_SMD:R_0805_2012Metric_Pad1.20x1.40mm_HandSolder
- added C10: 0.1uF, Capacitor_SMD:C_0805_2012Metric_Pad1.18x1.45mm_HandSolder, B.Cu at (138.9, 51.1)
- added C19: 0.1uF, Capacitor_SMD:C_0805_2012Metric_Pad1.18x1.45mm_HandSolder, B.Cu at (150.8, 42.2)
- added C20: 0.1uF, Capacitor_SMD:C_0805_2012Metric_Pad1.18x1.45mm_HandSolder, F.Cu at (140.3, 52.7)
- added C21: 1uF, Capacitor_SMD:C_0805_2012Metric_Pad1.18x1.45mm_HandSolder, F.Cu at (149.9, 47.8)
- added C22: 1uF, Capacitor_SMD:C_0805_2012Metric_Pad1.18x1.45mm_HandSolder, B.Cu at (148.7, 42.1)
- added C23: 1uF, Capacitor_SMD:C_0805_2012Metric_Pad1.18x1.45mm_HandSolder, F.Cu at (142.9, 52.7)
- added C24: 0.1uF, Capacitor_SMD:C_0805_2012Metric_Pad1.18x1.45mm_HandSolder, B.Cu at (150.6, 47.7)
- added C25: 1uF, Capacitor_SMD:C_0805_2012Metric_Pad1.18x1.45mm_HandSolder, B.Cu at (150.7, 45.4)
- added C26: 0.1uF, Capacitor_SMD:C_0805_2012Metric_Pad1.18x1.45mm_HandSolder, B.Cu at (147.6, 50.7)
- added C27: 0.1uF, Capacitor_SMD:C_0805_2012Metric_Pad1.18x1.45mm_HandSolder, B.Cu at (149.6, 50.6)
- added C28: 1uF, Capacitor_SMD:C_0805_2012Metric_Pad1.18x1.45mm_HandSolder, B.Cu at (145.6, 51.8)
- added C29: 1uF, Capacitor_SMD:C_0805_2012Metric_Pad1.18x1.45mm_HandSolder, B.Cu at (151.6, 50.7)
- added C5: 0.1uF, Capacitor_SMD:C_0805_2012Metric_Pad1.18x1.45mm_HandSolder, F.Cu at (147.2, 40.5)
- added C6: 0.1uF, Capacitor_SMD:C_0805_2012Metric_Pad1.18x1.45mm_HandSolder, F.Cu at (137.4, 52.3)
- added C8: 1uF, Capacitor_SMD:C_0805_2012Metric_Pad1.18x1.45mm_HandSolder, F.Cu at (147.2, 43.1)
- added C9: 1uF, Capacitor_SMD:C_0805_2012Metric_Pad1.18x1.45mm_HandSolder, F.Cu at (137.4, 49.7)
- added GND: MountingHole_3.2mm_M3_Pad, MountingHole:MountingHole_3.2mm_M3_Pad, F.Cu at (124.5, 33.0)
- added REF**: MountingHole_3.2mm_M3_Pad_TopBottom, MountingHole:MountingHole_3.2mm_M3_Pad_TopBottom, F.Cu at (124.5, 73.7)
- added REF**: MountingHole_3.2mm_M3_Pad_TopBottom, MountingHole:MountingHole_3.2mm_M3_Pad_TopBottom, F.Cu at (162.6, 73.7)
- added REF**: MountingHole_3.2mm_M3_Pad_TopBottom, MountingHole:MountingHole_3.2mm_M3_Pad_TopBottom, F.Cu at (162.6, 33.0)
- added TP1: TestPoint, TestPoint:TestPoint_Pad_D1.5mm, F.Cu at (157.5, 40.6)
- added TP10: TestPoint, TestPoint:TestPoint_Pad_D1.5mm, F.Cu at (157.5, 58.4)
- added TP11: TestPoint, TestPoint:TestPoint_Pad_D1.5mm, F.Cu at (134.6, 43.2)
- added TP12: TestPoint, TestPoint:TestPoint_Pad_D1.5mm, F.Cu at (157.5, 55.9)
- added TP13: TestPoint, TestPoint:TestPoint_Pad_D1.5mm, F.Cu at (157.5, 53.3)
- added TP14: TestPoint, TestPoint:TestPoint_Pad_D1.5mm, F.Cu at (129.5, 48.3)
- added TP15: TestPoint, TestPoint:TestPoint_Pad_D1.5mm, F.Cu at (129.5, 66.0)
- added TP16: TestPoint, TestPoint:TestPoint_Pad_D1.5mm, F.Cu at (151.7, 77.1)
- added TP17: TestPoint, TestPoint:TestPoint_Pad_D1.5mm, F.Cu at (142.5, 77.0)
- added TP18: TestPoint, TestPoint:TestPoint_Pad_D1.5mm, F.Cu at (129.5, 50.8)
- added TP19: TestPoint, TestPoint:TestPoint_Pad_D1.5mm, F.Cu at (129.5, 53.3)
- added TP2: TestPoint, TestPoint:TestPoint_Pad_D1.5mm, F.Cu at (157.5, 45.7)
- added TP20: TestPoint, TestPoint:TestPoint_Pad_D1.5mm, F.Cu at (129.5, 33.0)
- added TP21: TestPoint, TestPoint:TestPoint_THTPad_D1.5mm_Drill0.7mm, F.Cu at (136.7, 56.3)
- added TP22: TestPoint, TestPoint:TestPoint_THTPad_D1.5mm_Drill0.7mm, F.Cu at (129.5, 76.2)
- added TP23: TestPoint, TestPoint:TestPoint_Pad_D1.5mm, F.Cu at (146.6, 47.3)
- added TP24: TestPoint, TestPoint:TestPoint_THTPad_D1.5mm_Drill0.7mm, F.Cu at (160.0, 46.9)
- added TP25: TestPoint, TestPoint:TestPoint_THTPad_D1.5mm_Drill0.7mm, F.Cu at (157.5, 50.8)
- added TP3: TestPoint, TestPoint:TestPoint_Pad_D1.5mm, F.Cu at (129.5, 73.7)
- added TP4: TestPoint, TestPoint:TestPoint_Pad_D1.5mm, F.Cu at (157.5, 48.3)
- added TP5: TestPoint, TestPoint:TestPoint_Pad_D1.5mm, F.Cu at (157.5, 43.2)
- added TP6: TestPoint, TestPoint:TestPoint_Pad_D1.5mm, F.Cu at (151.6, 69.2)
- added TP7: TestPoint, TestPoint:TestPoint_Pad_D1.5mm, F.Cu at (129.5, 63.5)
- added TP8: TestPoint, TestPoint:TestPoint_Pad_D1.5mm, F.Cu at (157.5, 61.0)
- added TP9: TestPoint, TestPoint:TestPoint_Pad_D1.5mm, F.Cu at (157.5, 66.0)
- C1, U3: moved to F.Cu
- C16: value 4.7uF -> 1uF
- C18: value 47uf -> 0.1uF
- C7: renamed from C5; moved to F.Cu
- J3: value Electret Microphone -> Conn_01x02
- U4: value ADM7160ACPZN2.5-R7 -> AD7768-1BCPZ; footprint ADM7160ACPZN2-5-R7:CP_6_3_ADI -> AD7768:CP_28_12; moved to F.Cu
- U5: value LTC2508CDKD-32 -> ADXL359BCCZ; footprint Package_DFN_QFN:DFN-24-1EP_4x7mm_P0.5mm_EP2.64x6.44mm -> ADXL359:LGA14_CC-14-2_ADI; moved to B.Cu
- moved C7 18.1 mm to (151.7, 58.1), turned to 90 degrees
- moved C18 14.2 mm to (149.9, 45.3), turned to 0 degrees
- moved C16 14.0 mm to (136.4, 51.1), turned to -90 degrees
- moved C1 12.8 mm to (144.0, 58.1)
- moved U3 12.5 mm to (148.2, 57.7), turned to -90 degrees
- moved U4 10.1 mm to (142.2, 46.5)
- moved U5 4.96 mm to (146.1, 46.4), turned to -90 degrees
- moved C13 2.99 mm to (136.6, 70.8), turned to 0 degrees
- moved J2 2.54 mm to (132.1, 30.5)
- moved C11 0.67 mm to (140.4, 74.8)
- moved C12 0.67 mm to (142.9, 74.8)
- moved C14 0.67 mm to (137.8, 74.8)
- moved C15 0.67 mm to (135.3, 74.8)
- renumbered C6 to C11, C7 to C12, C8 to C13, C9 to C14, C10 to C15, C11 to C17
Connections:
- C16 pad 1: +5V -> Net-(U4-REGCAPA)
- C18 pad 1: REF -> Net-(U4-REGCAPD)
- J1 pad 12: G2 -> REF
- J1 pad 3: BUSY -> unconnected-(J1-SVP-Pad3)
- J1 pad 4: DRL -> unconnected-(J1-SVN-Pad4)
- J1 pad 5: SYNC -> ADC_DRDY*
- J1 pad 6: SEL1 -> ACCEL_DRDY
- J1 pad 7: SEL0 -> ACCEL_CS*
- J1 pad 8: REF -> ADC_SYNC
- J2 pad 10: unconnected-(J2-P5-Pad10) -> ADC_CS*
- J2 pad 13: +2V5 -> unconnected-(J2-P4-Pad13)
- J2 pad 15: unconnected-(J2-P2-Pad15) -> G2
- J2 pad 2: unconnected-(J2-P23-Pad2) -> MOSI_SPI
- J2 pad 6: unconnected-(J2-P21-Pad6) -> INT1
- J2 pad 8: SDOA -> MISO_SPI
- J2 pad 9: SCKA -> SCLK_SPI
- U4 pad 1: +2V5 -> +3.3V
- U4 pad 2: unconnected-(U4-NC-Pad2) -> ADC_SYNC
- U4 pad 3: GND -> unconnected-(U4-SYNC_OUT*-Pad3)
- U4 pad 4: +5V -> Net-(U4-REGCAPD)
- U4 pad 5: unconnected-(U4-NC-Pad5) -> +3.3V
- U4 pad 6: +5V -> +3.3V
- U5 pad 1: GND -> ACCEL_CS*
- U5 pad 10: REF -> Net-(U5-V1P8ANA)
- U5 pad 11: SEL0 -> +3.3V
- U5 pad 12: SEL1 -> INT1
- U5 pad 14: SYNC -> ACCEL_DRDY
- U5 pad 2: +3.3V -> SCLK_SPI
- U5 pad 3: +2V5 -> MOSI_SPI
- U5 pad 4: GND -> MISO_SPI
- U5 pad 5: Net-(U5-IN+) -> +3.3V
- U5 pad 6: Net-(U5-IN-) -> GND
- U5 pad 8: REF -> Net-(U5-V1P8DIG)
- U5 pad 9: REF -> GND
Routing:
- net REF: track 119.7 -> 67.2 mm, vias 2 -> 3
- net SDOA: track 50.7 -> 0.00 mm, vias 1 -> 0
- net SCKA: track 49.5 -> 0.00 mm, vias 1 -> 0
- net +2V5: track 46.3 -> 0.00 mm, vias 1 -> 0
- net SCLK_SPI: track 0.00 -> 41.7 mm, vias 0 -> 1
- net MISO_SPI: track 0.00 -> 40.0 mm, vias 0 -> 2
- net MOSI_SPI: track 0.00 -> 33.0 mm, vias 0 -> 3
- net MCLK: track 76.1 -> 43.3 mm
- net Net-(U5-IN-): track 29.0 -> 0.00 mm
- net ADC_DRDY*: track 0.00 -> 27.7 mm, vias 0 -> 1
- net ACCEL_DRDY: track 0.00 -> 27.1 mm
- net GND: track 99.1 -> 74.8 mm, vias 3 -> 10
- net ADC_CS*: track 0.00 -> 23.5 mm
- net Net-(U5-IN+): track 22.7 -> 0.00 mm
- net ACCEL_CS*: track 0.00 -> 21.5 mm, vias 0 -> 1
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- removed copper zone on In2.Cu, net GND
Other:
- board size 30.5 x 50.8 mm -> 48.3 x 50.8 mm
