File: pcb/ultrasonic_microphone.kicad_sch (KiCad schematic)
At the start: 33 parts, among them J1 Conn_01x19, J2 Conn_01x19, J3 Electret Microphone, U1 LTC6910-2CTS8-TRMPBF, U2 ADA4528-2ARMZ, U3 LTC6655CHMS8-3-PBF, U4 ADM7160ACPZN2.5-R7, U5 LTC2508CDKD-32

Commit message: Fabbed board
Parts:
- removed C12: 4.7uF, Capacitor_SMD:C_0805_2012Metric_Pad1.18x1.45mm_HandSolder, symbol Device:C
- removed C13, C14: 4.7uF, Capacitor_THT:C_Rect_L7.2mm_W7.2mm_P5.00mm_FKS2_FKP2_MKS2_MKP2, symbol Device:C
- removed C15: 10uF, Capacitor_SMD:C_0805_2012Metric_Pad1.18x1.45mm_HandSolder, symbol Device:C
- removed C17: 0.1uF, Capacitor_SMD:C_0805_2012Metric_Pad1.18x1.45mm_HandSolder, symbol Device:C
- removed R6, R7: 10, Resistor_SMD:R_0805_2012Metric_Pad1.20x1.40mm_HandSolder, symbol Device:R_US
- removed U4: ADM7160ACPZN2.5-R7, ADM7160ACPZN2-5-R7:CP_6_3_ADI, symbol ADM7160ACPZN2:ADM7160ACPZN2.5-R7
- removed U5: LTC2508CDKD-32, Package_DFN_QFN:DFN-24-1EP_4x7mm_P0.5mm_EP2.64x6.44mm, symbol Analog_ADC:LTC2508CDKD-32
- added C10, C19, C20, C24, C26, C27, C5, C6: 0.1uF, Capacitor_SMD:C_0805_2012Metric_Pad1.18x1.45mm_HandSolder, symbol Device:C
- added C21, C22, C23, C25, C28, C29, C8, C9: 1uF, Capacitor_SMD:C_0805_2012Metric_Pad1.18x1.45mm_HandSolder, symbol Device:C
- added TP1, TP10, TP11, TP12, TP13, TP14, TP15, TP16, TP17, TP18, TP19, TP2, TP20, TP21, TP22, TP23, TP24, TP25, TP3, TP4, TP5, TP6, TP7, TP8, TP9: TestPoint, TestPoint:TestPoint_Pad_D1.5mm, symbol Connector:TestPoint
- added U4: AD7768-1BCPZ, AD7768:CP_28_12, symbol AD7768:AD7768-1BCPZ
- added U5: ADXL359BCCZ, ADXL359:LGA14_CC-14-2_ADI, symbol ADXL359:ADXL359BCCZ
- C16: value 4.7uF -> 1uF
- C18: value 47uF -> 0.1uF
- J3: value Electret Microphone -> Conn_01x02
- renumbered C6 to C11, C7 to C12, C8 to C13, C9 to C14, C10 to C15, C11 to C17, C5 to C7
Connections:
- net +3.3V: now also C19.1, C22.1, C26.1, C28.1, C5.1, C6.1, C8.1, C9.1, U4.1 (RESET*), U4.22 (AVDD2), U4.5 (IOVDD), U4.6 (PIN*/SPI), U5.11 (VSUPPLY), U5.5 (VDDIO)
- net +5V: now also C20.2, C23.2, U4.23 (AVDD1); no longer C16.1
- net AMP_OUT: now also TP13.1, U4.27 (AIN+)
- net G0: now also TP9.1
- net G1: now also TP8.1
- net G2: now also J2.15 (P2), TP15.1; no longer J1.12 (P14)
- net GND: now also C10.2, C19.2, C20.1, C21.2, C22.2, C23.1, C24.2, C25.2, C26.2, C27.2, C28.2, C29.2, C5.2, C6.2, C8.2, C9.2, U4.13 (XTAL1), U4.21 (AVSS), U4.25 (REF-), U4.29 (EP(GND)), U4.7 (DGND), U4.8 (CLKSEL), U5.6 (VSSIO), U5.7 (RESERVED), U5.9 (VSS)
- net MCLK: now also TP7.1, U4.14 (MCLK/XTAL2), U5.13 (INT2)
- net REF: now also J1.12 (P14), TP10.1, U4.24 (REF+); no longer C18.1, J1.8 (P33)
- net VGND: now also TP12.1, U4.26 (AIN-)
- net at C4.1, R3.2, U1.3 (IN)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: now also TP6.1
- net at C4.2, R3.1, R4.1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: now also TP16.1
- net at C11.1, C12.1, C13.1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: now also TP17.1
- net at C11.2, C12.2, C13.2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: now also TP22.1
- net at R1.2, R2.1, U2.3 (INA+): now also TP3.1
- net ADC_CS*: now reaches J2.10 (P5)
- net ADC_CS*: now also TP19.1, U4.12 (CS*)
- net MOSI_SPI: now reaches J2.2 (P23)
- net MOSI_SPI: now also TP20.1, U4.11 (SDI), U5.3 (MOSI/SDA)
- net INT1: now reaches J2.6 (P21)
- net INT1: now also TP11.1, U5.12 (INT1)
- net +2V5: no longer names the net of J2.13 (P4)
- net BUSY: no longer names the net of J1.3 (SVP)
- net DRL: no longer names the net of J1.4 (SVN)
- net SCKA renamed SCLK_SPI
- net SCLK_SPI: now also TP18.1, U4.10 (SCLK), U5.2 (SCLK/VSSIO)
- net SDOA renamed MISO_SPI
- net MISO_SPI: now also TP14.1, U4.9 (DOUT/RDY*), U5.4 (MISO/ASEL)
- net SEL0 renamed ACCEL_CS*
- net ACCEL_CS*: now also TP2.1, U5.1 (*CS/SCL)
- net SEL1 renamed ACCEL_DRDY
- net ACCEL_DRDY: now also TP5.1, U5.14 (DRDY)
- net SYNC renamed ADC_DRDY*
- net ADC_DRDY*: now also TP1.1, U4.19 (DRDY*)
- new net: C10.1, C16.1, TP21.1, U4.20 (REGCAPA)
- new net: C18.1, C21.1, TP23.1, U4.4 (REGCAPD)
- new net: C24.1, C25.1, TP24.1, U5.8 (V1P8DIG)
- new net: C27.1, C29.1, TP25.1, U5.10 (V1P8ANA)
- new net ADC_SYNC: J1.8 (P33), TP4.1, U4.2 (SYNC_IN*)
- no-connect marks 22 -> 26
Other:
- moved on the sheet: J1, J2
